File: pcb/headphone.brd (EAGLE design)
At the start: 94 x 35.6 mm, 30 parts, among them IC101 LF353D, IC201 LF353N, IC301 LF353N, J101 MONOJACKSWITCHCRAFT3, J102 MONOJACKSWITCHCRAFT3, J201 MONOJACKNEUTRIK, J202 MONOJACKNEUTRIK, J301 STEREOJACK, J401 POWER_SIMPLE16, P101 DUALPOT 50K

Commit message: Panel!
Parts:
- moved R205 1.27 mm to (31.8, 15.2)
- moved R202 1.27 mm to (19.7, 14.0)
- moved J201 1.20 mm to (45.0, 11.0)
- moved J102 1.01 mm to (15.0, 8.00)
- moved P101 0.71 mm to (28.0, 8.00)
- moved J202 0.62 mm to (64.0, 11.0)
- moved J301 0.49 mm to (83.0, 11.0)
- moved J101 0.36 mm to (5.00, 8.00)
Routing:
- net N$12: track 2.67 -> 4.95 mm, vias 1 -> 0
- net N$3: track 17.2 -> 18.9 mm
- net N$10: track 26.9 -> 25.6 mm
- net J102: track 29.5 -> 30.4 mm
- net N$6: track 26.1 -> 26.9 mm
- net N$8: track 6.71 -> 6.02 mm
- net N$5: track 40.9 -> 41.4 mm

Commit message: fix for backwards volume knob and too-small text
Connections:
- removed net N$3 (its old number): J102.T, P101.D2
- new net N$5: J102.T, P101.U2
- net GND: now also P101.D1, P101.D2; no longer P101.U1, P101.U2
- net J102: now also P101.U1; no longer P101.D1
Routing:
- net N$3: track 41.4 -> 79.0 mm, vias 2 -> 0
- net N$3 (its old number): track 18.9 -> 0.00 mm
- net N$5: track 0.00 -> 11.5 mm
- net J102: track 30.4 -> 28.5 mm
- net N$2: track 26.9 -> 27.8 mm
