File: pcb/eurorack_headphones.kicad_pcb (KiCad board)
At the start: 2 copper layers, 97.5 x 41.5 mm, 30 parts, among them J101 JACK_2P, J102 JACK_2P, J201 JACK_2P, J202 JACK_2P, J301 JACK_TRS_6PINS, J401 EurorackPower, P101 POT_Dual 50k, U101 TL072, U201 TL072, U301 TL072

Commit message: Fix errors on board
Connections:
- J301 pad 1: Net-(J301-Pad1) -> GND
- J301 pad 2: GND -> Net-(J301-Pad2)
- R305 pad 1: Net-(J301-Pad1) -> Net-(J301-Pad2)
Routing:
- net /Left: track 40.8 -> 60.8 mm, vias 0 -> 2
- net Net-(J301-Pad1): track 19.0 -> 0.00 mm
- net GND: track 30.7 -> 44.6 mm, vias 1 -> 2
- net Net-(R301-Pad1): track 48.3 -> 35.4 mm
- net Net-(J301-Pad2): track 0.00 -> 6.29 mm
- net Net-(J301-Pad3): track 12.2 -> 16.7 mm
- net -12V: track 93.8 -> 95.5 mm
- net Net-(R203-Pad1): track 29.1 -> 30.3 mm
- net Net-(P101-Pad2): track 59.6 -> 60.7 mm
- net Net-(R201-Pad1): track 11.9 -> 12.9 mm
- net Net-(R302-Pad1): track 25.8 -> 26.7 mm
- net Net-(R202-Pad1): track 36.6 -> 37.3 mm
- net Net-(R204-Pad1): track 30.8 -> 31.4 mm
Other:
- net class Default: clearance 0.1524 -> 0.3
- rule trace_clearance: 0.1524 -> 0.3
- board text added: "Euro Amp v3.0 BY-CC-SA"
- board text removed: "Euro Amp v2.0 BY-CC-SA"
